File: Keyboard_PCB.kicad_sch (KiCad schematic)
At the start: 141 parts, among them U1 ESP32-WROOM-32E

Commit message: Finished Basic Keyboard Schematics
Connections:
- net Col 1: now also U1.26 (IO4)
- net Col 10: now also S10.1, S24.1, S38.1, S52.1, S66.1, U1.31 (IO19); no longer S21.1, S35.1, S49.1, S63.1, S7.1
- net Col 11: now also S11.1, S25.1, S39.1, S53.1, S67.1, U1.33 (IO21); no longer S22.1, S36.1, S50.1, S64.1, S8.1
- net Col 12: now also S12.1, S26.1, S40.1, S54.1, S68.1, U1.36 (IO22); no longer S23.1, S37.1, S51.1, S65.1, S9.1
- net Col 13: now also S13.1, S27.1, S41.1, S55.1, S69.1, U1.37 (IO23); no longer S10.1, S24.1, S38.1, S52.1, S66.1
- net Col 14: now also S14.1, S28.1, S42.1, S56.1, S70.1, U1.10 (IO25); no longer S11.1, S25.1, S39.1, S53.1, S67.1
- net Col 2: now also U1.29 (IO5)
- net Col 3: now also U1.14 (IO12)
- net Col 4: now also U1.16 (IO13)
- net Col 5: now also U1.13 (IO14)
- net Col 6: now also U1.23 (IO15)
- net Row 1: now also U1.11 (IO26)
- net Row 2: now also U1.12 (IO27)
- net Row 3: now also U1.8 (IO32)
- net Row 4: now also U1.9 (IO33)
- net Row 5: now also U1.6 (IO34)
- net Col 7: now reaches U1.27 (IO16)
- net Col 7: now also S21.1, S35.1, S49.1, S63.1, S7.1
- net Col 8: now reaches U1.28 (IO17)
- net Col 8: now also S22.1, S36.1, S50.1, S64.1, S8.1
- net Col 9: now reaches U1.30 (IO18)
- net Col 9: now also S23.1, S37.1, S51.1, S65.1, S9.1
